File: kicad_source/History.sch (KiCad schematic (older format))
At the start: 0 parts

Commit message: generated pdf files
Other:
- note added: "1.0"
- note added: "2019-12-31"
- note added: "Bernhard Mayer"
- note added: "initial release"
Changed lines of the file:
@@
 $Descr A4 11693 8268
 encoding utf-8
-Sheet 5 6
-Title ""
-Date ""
-Rev ""
-Comp ""
+Sheet 4 6
+Title "HighPowerMotorFeatherWing"
+Date "2019-12-31"
+Rev "1.0"
+Comp "generationmake"
 Comment1 ""
 Comment2 ""
 Comment3 ""
-Comment4 ""
+Comment4 "This documentation describes Open Hardware and is licensed under the CERN OHL v. 1.2."
 $EndDescr
+Text Notes 850  900  0    60   ~ 0
+1.0
+Text Notes 1350 900  0    60   ~ 0
+2019-12-31
+Text Notes 2300 900  0    60   ~ 0
+Bernhard Mayer
+Text Notes 3350 900  0    60   ~ 0
+initial release
 $EndSCHEMATC
